File: RTC-RV-3028-C7-breakout/RTC-RV-3028-C7-breakout.kicad_pcb (KiCad board)
At the start: 2 copper layers, 18.8 x 22.5 mm, 13 parts, among them J1 Conn_01x04_Female, J2 Conn_01x04_Female, U1 RV-3028-C7

Commit message: Fix mis-labeled components
Parts:
- removed MS621F: MS621F, Battery:BatteryHolder_Seiko_MS621F
- removed R1 DNP: 10k, Resistor_SMD:R_0603_1608Metric
- removed R7, R8: 10k, Resistor_SMD:R_0603_1608Metric
- added BT1: MS621F, Battery:BatteryHolder_Seiko_MS621F, F.Cu at (149.0, 96.1)
- added C1: 0.1µ, Capacitor_SMD:C_0603_1608Metric, F.Cu at (150.6, 91.0)
- added C2: 0.1µ, Capacitor_SMD:C_0603_1608Metric, F.Cu at (150.6, 87.8)
- added R1: 10k, Resistor_SMD:R_0603_1608Metric, B.Cu at (153.3, 88.8)
- R4, R5: value 0.1µ -> 10k
- moved R6 6.55 mm to (145.7, 87.8)
- moved R5 5.80 mm to (145.7, 91.1), turned to -90 degrees
- moved R4 3.76 mm to (152.3, 87.8), turned to 90 degrees
- moved R3 0.12 mm to (152.3, 91.0)
Connections:
- R4 pad 1: Net-(R3-Pad2) -> +3V3
- R4 pad 2: GND -> EVI
- R5 pad 1: +3V3 -> SDA
- R5 pad 2: GND -> +3V3
- R6 pad 1: +3V3 -> SCL
- R6 pad 2: EVI -> +3V3
Routing:
- net +3V3: track 30.5 -> 31.3 mm
